File: src_DTC-SVM/Three-phase_bridge/$Three-phase bridge.sch (KiCad schematic (older format))
At the start: 82 parts, among them M1 MCP6022-I/P, M2 MCP6022-I/P, P1 CONN_1, P2 POWER_FUSE, P4 CONN_1, P5 CONN_1, P6 POWER_FUSE, P7 CONN_1, P8 CONN_1, P9 CONN_1

Commit message: The wire up for the Three-phase bridge has been completed. Nevertheless, the fillzones still remain undone.
Changed lines of the file:
@@
 Connection ~ 2105 925
-$Comp
-L VCC #PWR070
-U 1 1 529AD657
-P 5580 455
-F 0 "#PWR070" H 5580 555 30  0001 C CNN
-F 1 "VCC" H 5580 555 30  0000 C CNN
-F 2 "" H 5580 455 60  0000 C CNN
-F 3 "" H 5580 455 60  0000 C CNN
-	1    5580 455
-	1    0    0    -1
-$EndComp
 $Comp
 L C C12
@@
 $EndComp
 $Comp
-L GND #PWR071
+L GND #PWR070
 U 1 1 529AD675
 P 5580 890
-F 0 "#PWR071" H 5580 890 30  0001 C CNN
+F 0 "#PWR070" H 5580 890 30  0001 C CNN
 F 1 "GND" H 5580 820 30  0001 C CNN
 F 2 "" H 5580 890 60  0000 C CNN
@@
 	5580 855  5580 890
 $Comp
-L +48V #PWR072
+L +48V #PWR071
 U 1 1 529C293E
 P 8840 2385
-F 0 "#PWR072" H 8840 2515 20  0001 C CNN
+F 0 "#PWR071" H 8840 2515 20  0001 C CNN
 F 1 "+48V" H 8840 2485 30  0000 C CNN
 F 2 "" H 8840 2385 60  0000 C CNN
@@
 	3310 4555 3310 4545
 $Comp
-L +48V #PWR073
+L +48V #PWR072
 U 1 1 529C34A5
 P -305 4940
-F 0 "#PWR073" H -305 5070 20  0001 C CNN
+F 0 "#PWR072" H -305 5070 20  0001 C CNN
 F 1 "+48V" H -305 5040 30  0000 C CNN
 F 2 "" H -305 4940 60  0000 C CNN
@@
 Wire Wire Line
 	-875 3135 -860 3135
+$Comp
+L +48V #PWR073
+U 1 1 529C4E46
+P 5580 455
+F 0 "#PWR073" H 5580 585 20  0001 C CNN
+F 1 "+48V" H 5580 555 30  0000 C CNN
+F 2 "" H 5580 455 60  0000 C CNN
+F 3 "" H 5580 455 60  0000 C CNN
+	1    5580 455
+	1    0    0    -1
+$EndComp
 $EndSCHEMATC
