File: src_DTC-SVM/Three-phase_bridge/Three-phase bridge.sch (KiCad schematic (older format))
At the start: 79 parts, among them K1 CONN_3, M1 MCP6022-I/P, M2 MCP6022-I/P, P1 CONN_1, P2 Fuse, P3 CONN_1, P4 CONN_1, P5 CONN_1, P6 CONN_2, SW1 SW_PUSH_SMALL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

Commit message: Kicad pcb has been separated into three bloks: stm32 connections, three-phase bridge and current sensing. The idea is to have the current operational and diffential amplifiers as close as possible to the shunt resistors and the stm32 pins so that there are no electromagnetic interferencies nor logs to the distance, specially because they are analog signals.
Parts:
- removed SW1, SW2, SW3, SW4, SW5, SW6: SW_PUSH_SMALL, ~, symbol SW_PUSH_SMALL
Connections:
- wire segments 130 -> 124
Changed lines of the file:
@@
 Wire Wire Line
 	4550 1000 4550 1035
-$Comp
-L SW_PUSH_SMALL SW1
-U 1 1 528ED996
-P 4740 1590
-F 0 "SW1" H 4890 1700 30  0000 C CNN
-F 1 "SW_PUSH_SMALL" H 4740 1511 30  0000 C CNN
-F 2 "~" H 4740 1590 60  0000 C CNN
-F 3 "~" H 4740 1590 60  0000 C CNN
-	1    4740 1590
-	1    0    0    -1
-$EndComp
-Wire Wire Line
-	4640 1490 4640 1370
-Connection ~ 4640 1370
-$Comp
-L VDD #PWR062
-U 1 1 528EDAF4
-P 4840 1690
-F 0 "#PWR062" H 4840 1790 30  0001 C CNN
-F 1 "VDD" H 4840 1800 30  0000 C CNN
-F 2 "" H 4840 1690 60  0000 C CNN
-F 3 "" H 4840 1690 60  0000 C CNN
-	1    4840 1690
-	-1   0    0    1
-$EndComp
-$Comp
-L SW_PUSH_SMALL SW4
-U 1 1 528EDBB1
-P 5555 4585
-F 0 "SW4" H 5705 4695 30  0000 C CNN
-F 1 "SW_PUSH_SMALL" H 5555 4506 30  0000 C CNN
-F 2 "~" H 5555 4585 60  0000 C CNN
-F 3 "~" H 5555 4585 60  0000 C CNN
-	1    5555 4585
-	1    0    0    -1
-$EndComp
-$Comp
-L VDD #PWR063
-U 1 1 528EDBB7
-P 5655 4685
-F 0 "#PWR063" H 5655 4785 30  0001 C CNN
-F 1 "VDD" H 5655 4795 30  0000 C CNN
-F 2 "" H 5655 4685 60  0000 C CNN
-F 3 "" H 5655 4685 60  0000 C CNN
-	1    5655 4685
-	-1   0    0    1
-$EndComp
-$Comp
-L SW_PUSH_SMALL SW2
-U 1 1 528EDBBD
-P 4035 1620
-F 0 "SW2" H 4185 1730 30  0000 C CNN
-F 1 "SW_PUSH_SMALL" H 4035 1541 30  0000 C CNN
-F 2 "~" H 4035 1620 60  0000 C CNN
-F 3 "~" H 4035 1620 60  0000 C CNN
-	1    4035 1620
-	1    0    0    -1
-$EndComp
-$Comp
-L VDD #PWR064
-U 1 1 528EDBC3
-P 4135 1720
-F 0 "#PWR064" H 4135 1820 30  0001 C CNN
-F 1 "VDD" H 4135 1830 30  0000 C CNN
-F 2 "" H 4135 1720 60  0000 C CNN
-F 3 "" H 4135 1720 60  0000 C CNN
-	1    4135 1720
-	-1   0    0    1
-$EndComp
-Wire Wire Line
-	3935 1520 3935 1170
-Connection ~ 3935 1170
-Wire Wire Line
-	5455 4485 5455 4345
-Connection ~ 5455 4345
-$Comp
-L SW_PUSH_SMALL SW6
-U 1 1 528EDE92
-P 5575 6130
-F 0 "SW6" H 5725 6240 30  0000 C CNN
-F 1 "SW_PUSH_SMALL" H 5575 6051 30  0000 C CNN
-F 2 "~" H 5575 6130 60  0000 C CNN
-F 3 "~" H 5575 6130 60  0000 C CNN
-	1    5575 6130
-	1    0    0    -1
-$EndComp
-$Comp
-L VDD #PWR065
-U 1 1 528EDE98
-P 5675 6230
-F 0 "#PWR065" H 5675 6330 30  0001 C CNN
-F 1 "VDD" H 5675 6340 30  0000 C CNN
-F 2 "" H 5675 6230 60  0000 C CNN
-F 3 "" H 5675 6230 60  0000 C CNN
-	1    5675 6230
-	-1   0    0    1
-$EndComp
-$Comp
-L SW_PUSH_SMALL SW5
-U 1 1 528EDE9E
-P 5605 5380
-F 0 "SW5" H 5755 5490 30  0000 C CNN
-F 1 "SW_PUSH_SMALL" H 5605 5301 30  0000 C CNN
-F 2 "~" H 5605 5380 60  0000 C CNN
-F 3 "~" H 5605 5380 60  0000 C CNN
-	1    5605 5380
-	1    0    0    -1
-$EndComp
-$Comp
-L VDD #PWR066
-U 1 1 528EDEA4
-P 5705 5480
-F 0 "#PWR066" H 5705 5580 30  0001 C CNN
-F 1 "VDD" H 5705 5590 30  0000 C CNN
-F 2 "" H 5705 5480 60  0000 C CNN
-F 3 "" H 5705 5480 60  0000 C CNN
-	1    5705 5480
-	-1   0    0    1
-$EndComp
-Wire Wire Line
-	5505 5280 5225 5280
 Connection ~ 5225 5280
 Wire Wire Line
-	5475 6030 5475 5935
-Connection ~ 5475 5935
-Wire Wire Line
 	2730 3855 5355 3855
-Wire Wire Line
-	5560 3790 5560 4145
-Connection ~ 5560 4145
 $Comp
 L LED D1
@@
 $EndComp
 $Comp
-L VCC #PWR067
+L VCC #PWR062
 U 1 1 528EE58C
 P 700 1495
-F 0 "#PWR067" H 700 1595 30  0001 C CNN
+F 0 "#PWR062" H 700 1595 30  0001 C CNN
 F 1 "VCC" H 700 1595 30  0000 C CNN
 F 2 "" H 700 1495 60  0000 C CNN
@@
 $EndComp
 $Comp
-L GND #PWR068
+L GND #PWR063
 U 1 1 528EE59B
 P 700 1895
-F 0 "#PWR068" H 700 1895 30  0001 C CNN
+F 0 "#PWR063" H 700 1895 30  0001 C CNN
 F 1 "GND" H 700 1825 30  0001 C CNN
 F 2 "" H 700 1895 60  0000 C CNN
@@
 $EndComp
 $Comp
-L VCC #PWR069
+L VCC #PWR064
 U 1 1 528EE91C
 P 615 2250
-F 0 "#PWR069" H 615 2350 30  0001 C CNN
+F 0 "#PWR064" H 615 2350 30  0001 C CNN
 F 1 "VCC" H 615 2350 30  0000 C CNN
 F 2 "" H 615 2250 60  0000 C CNN
@@
 $EndComp
 $Comp
-L SW_PUSH_SMALL SW3
-U 1 1 528F8A44
-P 5660 3890
-F 0 "SW3" H 5810 4000 30  0000 C CNN
-F 1 "SW_PUSH_SMALL" H 5660 3811 30  0000 C CNN
-F 2 "~" H 5660 3890 60  0000 C CNN
-F 3 "~" H 5660 3890 60  0000 C CNN
-	1    5660 3890
-	1    0    0    -1
-$EndComp
-$Comp
-L VDD #PWR070
-U 1 1 528F8A4A
-P 5760 3990
-F 0 "#PWR070" H 5760 4090 30  0001 C CNN
-F 1 "VDD" H 5760 4100 30  0000 C CNN
-F 2 "" H 5760 3990 60  0000 C CNN
-F 3 "" H 5760 3990 60  0000 C CNN
-	1    5760 3990
-	-1   0    0    1
-$EndComp
-$Comp
-L VDD #PWR071
+L VDD #PWR065
 U 1 1 528F8C0D
 P 4670 6315
-F 0 "#PWR071" H 4670 6415 30  0001 C CNN
+F 0 "#PWR065" H 4670 6415 30  0001 C CNN
 F 1 "VDD" H 4670 6425 30  0000 C CNN
 F 2 "" H 4670 6315 60  0000 C CNN
@@
 $EndComp
 $Comp
-L VDD #PWR072
+L VDD #PWR066
 U 1 1 528F8C1D
 P 1960 6275
-F 0 "#PWR072" H 1960 6375 30  0001 C CNN
+F 0 "#PWR066" H 1960 6375 30  0001 C CNN
 F 1 "VDD" H 1960 6385 30  0000 C CNN
 F 2 "" H 1960 6275 60  0000 C CNN
@@
 Connection ~ 8685 4115
 $Comp
-L +48V #PWR073
+L +48V #PWR067
 U 1 1 529384B4
 P 750 3050
-F 0 "#PWR073" H 750 3180 20  0001 C CNN
+F 0 "#PWR067" H 750 3180 20  0001 C CNN
 F 1 "+48V" H 750 3150 30  0000 C CNN
 F 2 "" H 750 3050 60  0000 C CNN
@@
 $EndComp
 $Comp
-L GND #PWR074
+L GND #PWR068
 U 1 1 52937FD5
 P 750 3650
-F 0 "#PWR074" H 750 3650 30  0001 C CNN
+F 0 "#PWR068" H 750 3650 30  0001 C CNN
 F 1 "GND" H 750 3580 30  0001 C CNN
 F 2 "" H 750 3650 60  0000 C CNN
@@
 $EndComp
 $Comp
-L +48V #PWR075
+L +48V #PWR069
 U 1 1 52938604
 P 8550 590
-F 0 "#PWR075" H 8550 720 20  0001 C CNN
+F 0 "#PWR069" H 8550 720 20  0001 C CNN
 F 1 "+48V" H 8550 690 30  0000 C CNN
 F 2 "" H 8550 590 60  0000 C CNN
@@
 $EndComp
 $Comp
-L +48V #PWR076
+L +48V #PWR070
 U 1 1 5293861A
 P 8370 3565
-F 0 "#PWR076" H 8370 3695 20  0001 C CNN
+F 0 "#PWR070" H 8370 3695 20  0001 C CNN
 F 1 "+48V" H 8370 3665 30  0000 C CNN
 F 2 "" H 8370 3565 60  0000 C CNN
@@
 $EndComp
 $Comp
-L +48V #PWR077
+L +48V #PWR071
 U 1 1 5293862E
 P 8370 5155
-F 0 "#PWR077" H 8370 5285 20  0001 C CNN
+F 0 "#PWR071" H 8370 5285 20  0001 C CNN
 F 1 "+48V" H 8370 5255 30  0000 C CNN
 F 2 "" H 8370 5155 60  0000 C CNN
@@
 $EndComp
 $Comp
-L +48V #PWR078
+L +48V #PWR072
 U 1 1 5293C7C4
 P 650 4050
-F 0 "#PWR078" H 650 4180 20  0001 C CNN
+F 0 "#PWR072" H 650 4180 20  0001 C CNN
 F 1 "+48V" H 650 4150 30  0000 C CNN
 F 2 "" H 650 4050 60  0000 C CNN
@@
 $EndComp
 $Comp
-L VCC #PWR079
+L VCC #PWR073
 U 1 1 5293C7DD
 P 650 4250
-F 0 "#PWR079" H 650 4350 30  0001 C CNN
+F 0 "#PWR073" H 650 4350 30  0001 C CNN
 F 1 "VCC" H 650 4350 30  0000 C CNN
 F 2 "" H 650 4250 60  0000 C CNN
@@
 $EndComp
 $Comp
-L +48V #PWR080
+L +48V #PWR074
 U 1 1 5293C863
 P 10135 5075
-F 0 "#PWR080" H 10135 5205 20  0001 C CNN
+F 0 "#PWR074" H 10135 5205 20  0001 C CNN
 F 1 "+48V" H 10135 5175 30  0000 C CNN
 F 2 "" H 10135 5075 60  0000 C CNN
@@
 $EndComp
 $Comp
-L +48V #PWR081
+L +48V #PWR075
 U 1 1 5293C895
 P 10245 3660
-F 0 "#PWR081" H 10245 3790 20  0001 C CNN
+F 0 "#PWR075" H 10245 3790 20  0001 C CNN
 F 1 "+48V" H 10245 3760 30  0000 C CNN
 F 2 "" H 10245 3660 60  0000 C CNN
@@
 $EndComp
 $Comp
-L +48V #PWR082
+L +48V #PWR076
 U 1 1 5293C8BD
 P 10620 585
-F 0 "#PWR082" H 10620 715 20  0001 C CNN
+F 0 "#PWR076" H 10620 715 20  0001 C CNN
 F 1 "+48V" H 10620 685 30  0000 C CNN
 F 2 "" H 10620 585 60  0000 C CNN

Commit message: Schematic and PCB updated.
Parts:
- added C10, C8: 0.1uF, ~, symbol C
- added C11: 0.33uF, ~, symbol C
- added C12, C13: 1000uF, ~, symbol C
- added C14, C15: 100uF, ~, symbol C
- added C9: 2.2uF, ~, symbol C
Connections:
- wire segments 124 -> 147
Other:
- moved on the sheet: LF1

Commit message: The wire up for the Three-phase bridge has been completed. Nevertheless, the fillzones still remain undone.
Parts:
- removed K1: CONN_3, ~, symbol CONN_3
- removed P2: Fuse, ~, symbol CONN_2
- removed P3: CONN_1, ~, symbol CONN_1
- removed P6: CONN_2, ~, symbol CONN_2
- added P2, P6: POWER_FUSE, ~, symbol POWER_FUSE
- added P7, P8, P9: CONN_1, ~, symbol CONN_1
Connections:
- wire segments 147 -> 159
- no-connect marks 48 -> 44
Other:
- moved on the sheet: BT1, BT2

Commit message: A couple of capacitors have been added to VDD, and a LED for the 48V signal (just for having a visual check).
Parts:
- added C16: 10uF, ~, symbol C
- added C17: 100uF, ~, symbol C
- added D5: LED, ~, symbol LED
Connections:
- wire segments 159 -> 162
Changed lines of the file:
@@
 $EndComp
 $Comp
-L GND #PWR071
+L GND #PWR070
 U 1 1 529AD675
 P 5580 890
-F 0 "#PWR071" H 5580 890 30  0001 C CNN
+F 0 "#PWR070" H 5580 890 30  0001 C CNN
 F 1 "GND" H 5580 820 30  0001 C CNN
 F 2 "" H 5580 890 60  0000 C CNN
@@
 	5580 855  5580 890
 $Comp
-L +48V #PWR072
+L +48V #PWR071
 U 1 1 529C293E
 P 8840 2385
-F 0 "#PWR072" H 8840 2515 20  0001 C CNN
+F 0 "#PWR071" H 8840 2515 20  0001 C CNN
 F 1 "+48V" H 8840 2485 30  0000 C CNN
 F 2 "" H 8840 2385 60  0000 C CNN
@@
 	3310 4555 3310 4545
 $Comp
-L +48V #PWR073
+L +48V #PWR072
 U 1 1 529C34A5
 P -305 4940
-F 0 "#PWR073" H -305 5070 20  0001 C CNN
+F 0 "#PWR072" H -305 5070 20  0001 C CNN
 F 1 "+48V" H -305 5040 30  0000 C CNN
 F 2 "" H -305 4940 60  0000 C CNN
@@
 	-875 3135 -860 3135
 $Comp
-L +48V #PWR?
+L +48V #PWR073
 U 1 1 529C4E46
 P 5580 455
-F 0 "#PWR?" H 5580 585 20  0001 C CNN
+F 0 "#PWR073" H 5580 585 20  0001 C CNN
 F 1 "+48V" H 5580 555 30  0000 C CNN
 F 2 "" H 5580 455 60  0000 C CNN
@@
 	1    0    0    -1
 $EndComp
+$Comp
+L C C16
+U 1 1 529C5E57
+P 4445 1745
+F 0 "C16" H 4445 1845 40  0000 L CNN
+F 1 "10uF" H 4451 1660 40  0000 L CNN
+F 2 "~" H 4483 1595 30  0000 C CNN
+F 3 "~" H 4445 1745 60  0000 C CNN
+	1    4445 1745
+	1    0    0    -1
+$EndComp
+$Comp
+L C C17
+U 1 1 529C5E5D
+P 4700 1745
+F 0 "C17" H 4700 1845 40  0000 L CNN
+F 1 "100uF" H 4706 1660 40  0000 L CNN
+F 2 "~" H 4738 1595 30  0000 C CNN
+F 3 "~" H 4700 1745 60  0000 C CNN
+	1    4700 1745
+	1    0    0    -1
+$EndComp
+$Comp
+L GND #PWR074
+U 1 1 529C5E63
+P 4445 1980
+F 0 "#PWR074" H 4445 1980 30  0001 C CNN
+F 1 "GND" H 4445 1910 30  0001 C CNN
+F 2 "" H 4445 1980 60  0000 C CNN
+F 3 "" H 4445 1980 60  0000 C CNN
+	1    4445 1980
+	1    0    0    -1
+$EndComp
+Wire Wire Line
+	4445 1945 4445 1980
+Wire Wire Line
+	4700 1545 4445 1545
+Wire Wire Line
+	4445 1945 4700 1945
+$Comp
+L VDD #PWR075
+U 1 1 529C5FF5
+P 4445 1545
+F 0 "#PWR075" H 4445 1645 30  0001 C CNN
+F 1 "VDD" H 4445 1655 30  0000 C CNN
+F 2 "" H 4445 1545 60  0000 C CNN
+F 3 "" H 4445 1545 60  0000 C CNN
+	1    4445 1545
+	1    0    0    -1
+$EndComp
+$Comp
+L LED D5
+U 1 1 529C678E
+P 745 2730
+F 0 "D5" H 745 2830 50  0000 C CNN
+F 1 "LED" H 745 2630 50  0000 C CNN
+F 2 "~" H 745 2730 60  0000 C CNN
+F 3 "~" H 745 2730 60  0000 C CNN
+	1    745  2730
+	0    1    1    0
+$EndComp
+$Comp
+L GND #PWR076
+U 1 1 529C679A
+P 745 2930
+F 0 "#PWR076" H 745 2930 30  0001 C CNN
+F 1 "GND" H 745 2860 30  0001 C CNN
+F 2 "" H 745 2930 60  0000 C CNN
+F 3 "" H 745 2930 60  0000 C CNN
+	1    745  2930
+	1    0    0    -1
+$EndComp
+$Comp
+L +48V #PWR077
+U 1 1 529C67A2
+P 745 2530
+F 0 "#PWR077" H 745 2660 20  0001 C CNN
+F 1 "+48V" H 745 2630 30  0000 C CNN
+F 2 "" H 745 2530 60  0000 C CNN
+F 3 "" H 745 2530 60  0000 C CNN
+	1    745  2530
+	1    0    0    -1
+$EndComp

Commit message: PCB is apparently completed. The connections, fillzones and screw holes are done in Kicad.
Parts:
- added P3: CONN_2, ~, symbol CONN_2
Changed lines of the file:
@@
+	1    0    0    -1
+$EndComp
+$Comp
+L +48V #PWR078
+U 1 1 529C7F85
+P -670 2420
+F 0 "#PWR078" H -670 2550 20  0001 C CNN
+F 1 "+48V" H -670 2520 30  0000 C CNN
+F 2 "" H -670 2420 60  0000 C CNN
+F 3 "" H -670 2420 60  0000 C CNN
+	1    -670 2420
+	1    0    0    -1
+$EndComp
+$Comp
+L VCC #PWR079
+U 1 1 529C7F94
+P -670 2620
+F 0 "#PWR079" H -670 2720 30  0001 C CNN
+F 1 "VCC" H -670 2720 30  0000 C CNN
+F 2 "" H -670 2620 60  0000 C CNN
+F 3 "" H -670 2620 60  0000 C CNN
+	1    -670 2620
+	1    0    0    -1
+$EndComp
+$Comp
+L CONN_2 P3
+U 1 1 529C7FF8
+P -320 2520
+F 0 "P3" V -370 2520 40  0000 C CNN
+F 1 "CONN_2" V -270 2520 40  0000 C CNN
+F 2 "~" H -320 2520 60  0000 C CNN
+F 3 "~" H -320 2520 60  0000 C CNN
+	1    -320 2520
 	1    0    0    -1
 $EndComp

Commit message: This is the PCB before editing the fill zones, the pads and clearance. The only inconsistency here is that the red Fill zones have chosen the wrong signals, so that the drain pins are not connected.
Parts:
- added STM32_CONN_Passive1: CONN_STM32_25X2_PASSIVE, ~, symbol CONN_STM32_25X2_PASSIVE
Connections:
- wire segments 162 -> 252
- no-connect marks 44 -> 16
Other:
- moved on the sheet: 1N1, 1N2, 1N3, BT1, BT2, C1, C10, C11, C12, C13, C14, C15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
