File: src_DTC-SVM/Three-phase_bridge/Three-phase bridge.sch (KiCad schematic (older format))
At the start: 87 parts, among them M1 MCP6022-I/P, M2 MCP6022-I/P, P1 CONN_1, P2 POWER_FUSE, P3 CONN_2, P4 CONN_1, P5 CONN_1, P6 POWER_FUSE, P7 CONN_1, P8 CONN_1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

Commit message: PCB: the hall-effect current sensors have been added. Python: multiple graphics have been enabled within a figure
Parts:
- added ACS1, ACS2: ACS712, ~, symbol ACS712
- added C18, C20: 0.1uF, ~, symbol C
- added C19, C21: 1nF, ~, symbol C
Connections:
- wire segments 252 -> 309
