File: src_DTC-SVM/Three-phase_bridge/_autosave-Three-phase bridge.kicad_pcb (KiCad board)
At the start: 2 copper layers, 419.1 x 318 mm, 101 parts, among them M1 MCP6022-I/P, M2 MCP6022-I/P, P1 CONN_1, P2 POWER_FUSE, P3 CONN_2, P4 CONN_1, P5 CONN_1, P6 POWER_FUSE, P7 CONN_1, P8 CONN_1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

Commit message: Python file can now receive from and transmit to the stm32f4, as well as print, save in a file, and plot such data. The python code has also been split into three files.
Parts:
- removed ACS1, ACS2: ACS712, ACS712
- removed C18, C20: 0.1uF, 6mm_C
- removed C19, C21: 1nF, 6mm_C
Routing:
- added copper zone on F.Cu, net N-000006
- added copper zone on F.Cu, net N-0000061
- added copper zone on F.Cu, net N-0000062
- removed copper zone on F.Cu, net N-000003
- removed copper zone on F.Cu, net N-0000055
- removed copper zone on F.Cu, net N-0000058
