File: src_DTC-SVM/Three-phase_bridge_SMD/Three-phase bridge.sch (KiCad schematic (older format))
At the start: 93 parts, among them M1 MCP6022-I/P, M2 MCP6022-I/P, P1 CONN_1, P2 POWER_FUSE, P3 CONN_2, P4 CONN_1, P5 CONN_1, P6 POWER_FUSE, P7 CONN_1, P8 CONN_1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

Commit message: PCB: All resistances and most of capacitors have been replaced by their SMD counter parts. Required space have been sustancially reduced.
Parts:
- removed P7, P8, P9: CONN_1, ~, symbol CONN_1
Connections:
- wire segments 309 -> 302
Changed lines of the file:
@@
-$EndComp
-$Comp
-L CONN_STM32_25X2 STM32_CONN1
-U 1 1 528E7B9F
-P 3080 3500
-F 0 "STM32_CONN1" H 3180 4700 60  0000 C CNN
-F 1 "CONN_STM32_25X2" H 3180 2000 50  0000 C CNN
-F 2 "~" H 3030 3100 60  0000 C CNN
-F 3 "~" H 3030 3100 60  0000 C CNN
-	1    3080 3500
-	1    0    0    -1
 $EndComp
 $Comp
@@
 $EndComp
 $Comp
-L CONN_1 P7
-U 1 1 529C2CCE
-P 4455 4355
-F 0 "P7" H 4535 4355 40  0000 L CNN
-F 1 "CONN_1" H 4455 4410 30  0001 C CNN
-F 2 "~" H 4455 4355 60  0000 C CNN
-F 3 "~" H 4455 4355 60  0000 C CNN
-	1    4455 4355
-	1    0    0    -1
-$EndComp
-$Comp
-L CONN_1 P8
-U 1 1 529C2CD4
-P 4455 4445
-F 0 "P8" H 4535 4445 40  0000 L CNN
-F 1 "CONN_1" H 4455 4500 30  0001 C CNN
-F 2 "~" H 4455 4445 60  0000 C CNN
-F 3 "~" H 4455 4445 60  0000 C CNN
-	1    4455 4445
-	1    0    0    -1
-$EndComp
-$Comp
-L CONN_1 P9
-U 1 1 529C2CDA
-P 4460 4540
-F 0 "P9" H 4540 4540 40  0000 L CNN
-F 1 "CONN_1" H 4460 4595 30  0001 C CNN
-F 2 "~" H 4460 4540 60  0000 C CNN
-F 3 "~" H 4460 4540 60  0000 C CNN
-	1    4460 4540
-	1    0    0    -1
-$EndComp
-$Comp
 L +48V #PWR071
 U 1 1 529C34A5
@@
 	6580 850  6580 885
 Wire Wire Line
-	3730 4350 4285 4350
-Wire Wire Line
-	4285 4350 4285 4355
-Wire Wire Line
-	4285 4355 4305 4355
-Wire Wire Line
-	4305 4445 3730 4445
-Wire Wire Line
-	3730 4445 3730 4450
-Wire Wire Line
-	3730 4550 4310 4550
-Wire Wire Line
-	4310 4550 4310 4540
-Wire Wire Line
 	1615 -550 1845 -550
 Wire Wire Line
@@
 Wire Wire Line
 	3730 4355 3730 4350
-Wire Wire Line
-	3730 4450 825  4450
-Wire Wire Line
-	825  4450 825  4455
 Wire Wire Line
 	825  4555 3730 4555
@@
 Wire Wire Line
 	1675 5315 2485 5315
+$Comp
+L CONN_STM32_25X2 STM32_CONN1
+U 1 1 528E7B9F
+P 3080 3500
+F 0 "STM32_CONN1" H 3180 4700 60  0000 C CNN
+F 1 "CONN_STM32_25X2" H 3180 2000 50  0000 C CNN
+F 2 "~" H 3030 3100 60  0000 C CNN
+F 3 "~" H 3030 3100 60  0000 C CNN
+	1    3080 3500
+	1    0    0    -1
+$EndComp
+Wire Wire Line
+	825  4455 3730 4455
+Wire Wire Line
+	3730 4455 3730 4450
 $EndSCHEMATC

Commit message: Changing leds to SMD.
Parts:
- added R27, R28: R, ~, symbol R
Connections:
- wire segments 302 -> 307
Changed lines of the file:
@@
 Sheet 1 1
 Title ""
-Date "17 dec 2013"
+Date "19 dec 2013"
 Rev ""
 Comp ""
@@
 L GND #PWR058
 U 1 1 528EE59B
-P 3250 -260
-F 0 "#PWR058" H 3250 -260 30  0001 C CNN
-F 1 "GND" H 3250 -330 30  0001 C CNN
-F 2 "" H 3250 -260 60  0000 C CNN
-F 3 "" H 3250 -260 60  0000 C CNN
-	1    3250 -260
+P 3185 265
+F 0 "#PWR058" H 3185 265 30  0001 C CNN
+F 1 "GND" H 3185 195 30  0001 C CNN
+F 2 "" H 3185 265 60  0000 C CNN
+F 3 "" H 3185 265 60  0000 C CNN
+	1    3185 265
 	1    0    0    -1
 $EndComp
@@
 L GND #PWR075
 U 1 1 529C679A
-P 2645 -225
-F 0 "#PWR075" H 2645 -225 30  0001 C CNN
-F 1 "GND" H 2645 -295 30  0001 C CNN
-F 2 "" H 2645 -225 60  0000 C CNN
-F 3 "" H 2645 -225 60  0000 C CNN
-	1    2645 -225
-	1    0    0    -1
+P 2110 -225
+F 0 "#PWR075" H 2110 -225 30  0001 C CNN
+F 1 "GND" H 2110 -295 30  0001 C CNN
+F 2 "" H 2110 -225 60  0000 C CNN
+F 3 "" H 2110 -225 60  0000 C CNN
+	1    2110 -225
+	0    1    1    0
 $EndComp
 $Comp
@@
 Wire Wire Line
 	3730 4455 3730 4450
+$Comp
+L R R27
+U 1 1 52B244CC
+P 2370 -225
+F 0 "R27" V 2450 -225 40  0000 C CNN
+F 1 "R" V 2377 -224 40  0000 C CNN
+F 2 "~" V 2300 -225 30  0000 C CNN
+F 3 "~" H 2370 -225 30  0000 C CNN
+	1    2370 -225
+	0    -1   -1   0
+$EndComp
+Wire Wire Line
+	2120 -225 2110 -225
+Wire Wire Line
+	2620 -225 2645 -225
+$Comp
+L R R28
+U 1 1 52B2479C
+P 3185 -5
+F 0 "R28" V 3265 -5  40  0000 C CNN
+F 1 "R" V 3192 -4  40  0000 C CNN
+F 2 "~" V 3115 -5  30  0000 C CNN
+F 3 "~" H 3185 -5  30  0000 C CNN
+	1    3185 -5
+	1    0    0    -1
+$EndComp
+Wire Wire Line
+	3250 -260 3185 -260
+Wire Wire Line
+	3185 -260 3185 -255
+Wire Wire Line
+	3185 245  3185 265
 $EndSCHEMATC

Commit message: Fueses have been converted to SMD. THE ACS712/ACS714 have been wired.
Connections:
- wire segments 307 -> 302
Other:
- moved on the sheet: P1, P4
Changed lines of the file:
@@
 L CONN_1 P1
 U 1 1 528E8620
-P 11980 1135
-F 0 "P1" H 12060 1135 40  0000 L CNN
-F 1 "CONN_1" H 11980 1190 30  0001 C CNN
-F 2 "~" H 11980 1135 60  0000 C CNN
-F 3 "~" H 11980 1135 60  0000 C CNN
-	1    11980 1135
+P 12145 740
+F 0 "P1" H 12225 740 40  0000 L CNN
+F 1 "CONN_1" H 12145 795 30  0001 C CNN
+F 2 "~" H 12145 740 60  0000 C CNN
+F 3 "~" H 12145 740 60  0000 C CNN
+	1    12145 740
 	1    0    0    -1
 $EndComp
@@
 L CONN_1 P4
 U 1 1 528E8B36
-P 11800 4110
-F 0 "P4" H 11880 4110 40  0000 L CNN
-F 1 "CONN_1" H 11800 4165 30  0001 C CNN
-F 2 "~" H 11800 4110 60  0000 C CNN
-F 3 "~" H 11800 4110 60  0000 C CNN
-	1    11800 4110
+P 12390 3870
+F 0 "P4" H 12470 3870 40  0000 L CNN
+F 1 "CONN_1" H 12390 3925 30  0001 C CNN
+F 2 "~" H 12390 3870 60  0000 C CNN
+F 3 "~" H 12390 3870 60  0000 C CNN
+	1    12390 3870
 	1    0    0    -1
 $EndComp
@@
 $EndComp
 $Comp
-L ACS712 ACS1
-U 1 1 52A8F3FC
-P 12800 1150
-F 0 "ACS1" H 12820 900 60  0000 C CNN
-F 1 "ACS712" H 12820 1500 60  0000 C CNN
-F 2 "~" H 12820 1500 60  0000 C CNN
-F 3 "~" H 12820 1500 60  0000 C CNN
-	1    12800 1150
-	1    0    0    -1
-$EndComp
-$Comp
 L +5V #PWR084
 U 1 1 52A8FC3A
@@
 Wire Wire Line
 	11150 4405 10920 4405
-Wire Wire Line
-	11150 3935 11150 4405
 Connection ~ 9370 4110
 Wire Wire Line
@@
 Wire Wire Line
 	11330 1430 11100 1430
-Wire Wire Line
-	11330 935  11330 1430
 Connection ~ 9550 1135
 Wire Wire Line
@@
 Wire Wire Line
 	9685 3770 9685 4110
-Connection ~ 11650 4110
 Wire Wire Line
 	10060 695  10060 1135
@@
 Connection ~ 9685 4110
 Wire Wire Line
-	11830 1135 11830 1530
-Wire Wire Line
 	3900 945  3900 865
 Wire Wire Line
@@
 	825  2550 825  2555
 Wire Wire Line
-	11650 3985 11650 4505
-Wire Wire Line
-	11330 935  12320 935
-Wire Wire Line
-	12320 935  12320 1000
-Connection ~ 11330 1135
-Wire Wire Line
-	12320 1100 12290 1100
-Wire Wire Line
-	12290 1100 12290 1000
-Wire Wire Line
-	12290 1000 12320 1000
-Wire Wire Line
 	12320 1200 12285 1200
 Wire Wire Line
@@
 	12285 1300 12320 1300
 Wire Wire Line
-	11830 1250 11830 1245
-Wire Wire Line
-	11830 1245 12285 1245
-Connection ~ 12285 1245
-Connection ~ 11830 1250
-Wire Wire Line
 	13320 1300 13320 1340
 Wire Wire Line
@@
 	13195 4510 13230 4510
 Wire Wire Line
-	11725 4455 13195 4455
-Connection ~ 13195 4455
-Wire Wire Line
 	14230 4510 14230 4550
 Wire Wire Line
@@
 	14930 4310 14230 4310
 Wire Wire Line
-	11150 3935 12240 3935
-Wire Wire Line
-	12240 3935 12240 4145
-Connection ~ 11150 4110
-Wire Wire Line
-	11725 4455 11725 4280
-Wire Wire Line
-	11725 4280 11650 4280
-Connection ~ 11650 4280
-Wire Wire Line
-	11650 3985 11685 3985
-Wire Wire Line
-	11685 3985 11685 4110
-Wire Wire Line
-	11685 4110 11650 4110
+	12240 3870 12240 4145
 Wire Wire Line
 	14930 4310 14930 8325
@@
 Wire Wire Line
 	3185 245  3185 265
+Wire Wire Line
+	11330 1135 11330 1430
+$Comp
+L ACS712 ACS1
+U 1 1 52A8F3FC
+P 12800 1150
+F 0 "ACS1" H 12820 900 60  0000 C CNN
+F 1 "ACS712" H 12820 1500 60  0000 C CNN
+F 2 "~" H 12820 1500 60  0000 C CNN
+F 3 "~" H 12820 1500 60  0000 C CNN
+	1    12800 1150
+	1    0    0    -1
+$EndComp
+Wire Wire Line
+	12320 1000 12320 1100
+Wire Wire Line
+	11830 1135 11830 1530
+Wire Wire Line
+	11830 1135 12240 1135
+Wire Wire Line
+	12240 1135 12240 1265
+Wire Wire Line
+	12240 1265 12285 1265
+Connection ~ 12285 1265
+Wire Wire Line
+	12320 1050 11995 1050
+Wire Wire Line
+	11995 1050 11995 740
+Connection ~ 12320 1050
+Wire Wire Line
+	11150 4110 11150 4405
+Wire Wire Line
+	11650 4505 11650 4110
+Wire Wire Line
+	11650 4110 12145 4110
+Wire Wire Line
+	12145 4110 12145 4455
+Wire Wire Line
+	12145 4455 13195 4455
+Connection ~ 13195 4455
 $EndSCHEMATC

Commit message: New ADC ports for the hall current sensors have been added to the PCB. Rewiring of surrounding connections is being carried out.
Connections:
- wire segments 302 -> 297
Changed lines of the file:
@@
 Sheet 1 1
 Title ""
-Date "19 dec 2013"
+Date "12 jan 2014"
 Rev ""
 Comp ""
@@
 	825  2650 825  2655
 Wire Wire Line
-	825  2755 3730 2755
-Wire Wire Line
-	3730 2755 3730 2750
-Wire Wire Line
-	3730 2850 825  2850
-Wire Wire Line
-	825  2850 825  2855
+	3730 2755 825  2755
+Wire Wire Line
+	3730 1985 3730 2755
+Wire Wire Line
+	825  2815 825  2855
 Wire Wire Line
 	825  2955 3730 2955
@@
 	13600 600  13440 600
 Wire Wire Line
-	8910 2845 9160 2845
-Wire Wire Line
-	9160 2845 9160 2190
-Wire Wire Line
-	9160 2190 14020 2190
-Wire Wire Line
-	14020 2190 14020 1100
-Wire Wire Line
-	14020 1100 13320 1100
-Wire Wire Line
 	12240 4145 13230 4145
 Wire Wire Line
@@
 	14510 3810 14350 3810
 Wire Wire Line
-	14930 4310 14230 4310
-Wire Wire Line
 	12240 3870 12240 4145
-Wire Wire Line
-	14930 4310 14930 8325
-Wire Wire Line
-	14930 8325 1685 8325
-Wire Wire Line
-	1685 8325 1685 5405
-Wire Wire Line
-	1685 5405 1675 5405
-Wire Wire Line
-	2485 5315 2485 3060
 Connection ~ 2485 3060
-Wire Wire Line
-	1675 5405 1675 5315
-Wire Wire Line
-	1675 5315 2485 5315
 $Comp
 L CONN_STM32_25X2 STM32_CONN1
@@
 	12145 4455 13195 4455
 Connection ~ 13195 4455
+Wire Wire Line
+	3730 1985 13790 1985
+Wire Wire Line
+	13790 1985 13790 1100
+Wire Wire Line
+	13790 1100 13320 1100
+Connection ~ 3730 2750
+Wire Wire Line
+	2630 2035 2630 2850
+Wire Wire Line
+	2630 2035 14610 2035
+Wire Wire Line
+	14610 2035 14610 4310
+Wire Wire Line
+	14610 4310 14230 4310
+Connection ~ 2630 2850
+Wire Wire Line
+	3730 2850 3730 2815
+Wire Wire Line
+	3730 2815 825  2815
 $EndSCHEMATC

Commit message: PCB holes and fillzones fixed on the Three-phase_bridge_SMD design.
Parts:
- removed RGL1, RGL2, RGL3: RG_LED, ~, symbol RG_LED
- added D10, D11, D6, D7, D8, D9: LED, ~, symbol LED
- added RV1, RV2, RV3, RV4: POT, ~, symbol POT
Connections:
- wire segments 297 -> 327
- no-connect marks 16 -> 20
