File: src_DTC-SVM/bigger_tracks_Three-phase_bridge_SMD/$Three-phase bridge.sch (KiCad schematic (older format))
At the start: 105 parts, among them M1 MCP6022-I/P, M2 MCP6022-I/P, P1 CONN_1, P2 POWER_FUSE, P3 CONN_2, P4 CONN_1, P5 CONN_1, P6 POWER_FUSE

Commit message: The PCB has been updated with wider tracks and pads (0.097 in, the maximum value before they touch each other).
Parts:
- gave numbers to parts that had none: 7
Changed lines of the file:
@@
 	3730 2500 3730 2550
 $Comp
-L CONN_1 P?
+L CONN_1 P12
 U 1 1 5305553B
 P 14100 5750
-F 0 "P?" H 14180 5750 40  0000 L CNN
+F 0 "P12" H 14180 5750 40  0000 L CNN
 F 1 "CONN_1" H 14100 5805 30  0001 C CNN
 F 2 "" H 14100 5750 60  0000 C CNN
@@
 $EndComp
 $Comp
-L CONN_1 P?
+L CONN_1 P7
 U 1 1 5305554A
 P 14050 6100
-F 0 "P?" H 14130 6100 40  0000 L CNN
+F 0 "P7" H 14130 6100 40  0000 L CNN
 F 1 "CONN_1" H 14050 6155 30  0001 C CNN
 F 2 "" H 14050 6100 60  0000 C CNN
@@
 $EndComp
 $Comp
-L CONN_1 P?
+L CONN_1 P8
 U 1 1 53055559
 P 14050 6400
-F 0 "P?" H 14130 6400 40  0000 L CNN
+F 0 "P8" H 14130 6400 40  0000 L CNN
 F 1 "CONN_1" H 14050 6455 30  0001 C CNN
 F 2 "" H 14050 6400 60  0000 C CNN
@@
 $EndComp
 $Comp
-L CONN_1 P?
+L CONN_1 P9
 U 1 1 53055568
 P 14050 6750
-F 0 "P?" H 14130 6750 40  0000 L CNN
+F 0 "P9" H 14130 6750 40  0000 L CNN
 F 1 "CONN_1" H 14050 6805 30  0001 C CNN
 F 2 "" H 14050 6750 60  0000 C CNN
@@
 $EndComp
 $Comp
-L CONN_1 P?
+L CONN_1 P10
 U 1 1 53055577
 P 14050 6950
-F 0 "P?" H 14130 6950 40  0000 L CNN
+F 0 "P10" H 14130 6950 40  0000 L CNN
 F 1 "CONN_1" H 14050 7005 30  0001 C CNN
 F 2 "" H 14050 6950 60  0000 C CNN
@@
 $EndComp
 $Comp
-L CONN_1 P?
+L CONN_1 P11
 U 1 1 53055586
 P 14050 7300
-F 0 "P?" H 14130 7300 40  0000 L CNN
+F 0 "P11" H 14130 7300 40  0000 L CNN
 F 1 "CONN_1" H 14050 7355 30  0001 C CNN
 F 2 "" H 14050 7300 60  0000 C CNN
@@
 $EndComp
 $Comp
-L CONN_1 P?
+L CONN_1 P13
 U 1 1 53055595
 P 14100 7600
-F 0 "P?" H 14180 7600 40  0000 L CNN
+F 0 "P13" H 14180 7600 40  0000 L CNN
 F 1 "CONN_1" H 14100 7655 30  0001 C CNN
 F 2 "" H 14100 7600 60  0000 C CNN
