File: src_DTC-SVM/bigger_tracks_Three-phase_bridge_SMD/Three-phase bridge.sch (KiCad schematic (older format))
At the start: 105 parts, among them M1 MCP6022-I/P, M2 MCP6022-I/P, P1 CONN_1, P10 CONN_1, P11 CONN_1, P12 CONN_1, P13 CONN_1, P2 POWER_FUSE, P3 CONN_2, P4 CONN_1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

Commit message: PCB: Fixed missing connection between pins 5 from the IRF2110 to the shunt resistors. The pdf generation for the laser cutter is still pending.
Connections:
- wire segments 244 -> 262
Changed lines of the file:
@@
 Sheet 1 1
 Title ""
-Date "20 feb 2014"
+Date "24 mar 2014"
 Rev ""
 Comp ""
@@
 NoConn ~ 13900 7300
 NoConn ~ 13950 7600
+Wire Wire Line
+	8310 1165 8310 1215
+Wire Wire Line
+	8310 1215 8440 1215
+Wire Wire Line
+	8440 1215 8440 1310
+Wire Wire Line
+	8440 1310 9495 1310
+Wire Wire Line
+	9495 1310 9495 1190
+Wire Wire Line
+	9495 1190 9550 1190
+Connection ~ 9550 1190
+Wire Wire Line
+	8130 4140 8130 4200
+Wire Wire Line
+	8130 4200 8250 4200
+Wire Wire Line
+	8250 4200 8250 4280
+Wire Wire Line
+	8250 4280 8910 4280
+Wire Wire Line
+	8910 4280 8910 4200
+Wire Wire Line
+	8910 4200 9370 4200
+Connection ~ 9370 4200
+Wire Wire Line
+	8130 5730 8130 5780
+Wire Wire Line
+	8130 5780 8260 5780
+Wire Wire Line
+	8260 5780 8260 5890
+Wire Wire Line
+	8260 5890 8925 5890
+Wire Wire Line
+	8925 5890 8925 5835
+Wire Wire Line
+	8925 5835 9370 5835
+Connection ~ 9370 5835
 $EndSCHEMATC
