File: src_DTC-SVM/bigger_tracks_Three-phase_bridge_SMD/_autosave-Three-phase bridge.kicad_pcb (KiCad board)
At the start: 2 copper layers, 401.6 x 318 mm, 105 parts, among them M1 MCP6022-I/P, M2 MCP6022-I/P, P1 CONN_1, P10 CONN_1, P11 CONN_1, P12 CONN_1, P13 CONN_1, P2 POWER_FUSE, P3 CONN_2, P4 CONN_1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

Commit message: Testing code for designing LPF with python.
Other:
- net class Default: trace_width 7.62 -> 0.508
Changed lines of the file:
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@@
   (layers
     (15 F.Cu signal)
-    (0 B.Cu signal hide)
+    (0 B.Cu signal)
     (16 B.Adhes user)
     (17 F.Adhes user)
@@
   )
   (setup
-    (last_trace_width 7.62)
+    (last_trace_width 0.508)
     (user_trace_width 1.143)
     (user_trace_width 1.2192)
@@
   (net_class Default "This is the default net class."
     (clearance 0.0254)
-    (trace_width 7.62)
+    (trace_width 0.508)
     (via_dia 0.127)
     (via_drill 0.1016)

Commit message: After having changed the PCB to handle 56V instead of 12V.
Other:
- net class Default: trace_width 0.508 -> 7.62
Changed lines of the file:
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@@
   (layers
     (15 F.Cu signal)
-    (0 B.Cu signal)
+    (0 B.Cu signal hide)
     (16 B.Adhes user)
     (17 F.Adhes user)
@@
   )
   (setup
-    (last_trace_width 0.508)
+    (last_trace_width 7.62)
     (user_trace_width 1.143)
     (user_trace_width 1.2192)
@@
   (net_class Default "This is the default net class."
     (clearance 0.0254)
-    (trace_width 0.508)
+    (trace_width 7.62)
     (via_dia 0.127)
     (via_drill 0.1016)
