File: src_PCB_Mobile_base/Three-phase bridge.sch (KiCad schematic (older format))
At the start: 105 parts, among them M1 MCP6022-I/P, M2 MCP6022-I/P, P1 CONN_1, P10 CONN_1, P11 CONN_1, P12 CONN_1, P13 CONN_1, P2 POWER_FUSE, P3 CONN_2, P4 CONN_1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

Commit message: Eliminacion de conecciones de Pin 8 y 9 del stm 32
Parts:
- removed ACS1, ACS2: ACS712, ~, symbol ACS712
- removed C18, C20: 0.1uF, ~, symbol C
- removed C19, C21: 1nF, ~, symbol C
Connections:
- wire segments 262 -> 215
- no-connect marks 56 -> 58
Other:
- moved on the sheet: P1, P4

Commit message: se agrego _autosave* al gitignore y se eliminaron los potenciometros
Parts:
- removed RV1, RV2, RV3, RV4: POT, ~, symbol POT
Connections:
- wire segments 215 -> 200
- no-connect marks 58 -> 54

Commit message: PCB potencia y PCB resolver version de Philip Koenig
Parts:
- removed P11, P12, P13: CONN_1, symbol CONN_1
Connections:
- no-connect marks 54 -> 51
Changed lines of the file:
@@
 Sheet 1 1
 Title ""
-Date "30 sep 2014"
+Date "16 oct 2014"
 Rev ""
 Comp ""
@@
 	3730 2500 3730 2550
 $Comp
-L CONN_1 P12
-U 1 1 5305553B
-P 14100 5750
-F 0 "P12" H 14180 5750 40  0000 L CNN
-F 1 "CONN_1" H 14100 5805 30  0001 C CNN
-F 2 "" H 14100 5750 60  0000 C CNN
-F 3 "" H 14100 5750 60  0000 C CNN
-	1    14100 5750
-	1    0    0    -1
-$EndComp
-$Comp
-L CONN_1 P7
-U 1 1 5305554A
-P 14050 6100
-F 0 "P7" H 14130 6100 40  0000 L CNN
-F 1 "CONN_1" H 14050 6155 30  0001 C CNN
-F 2 "" H 14050 6100 60  0000 C CNN
-F 3 "" H 14050 6100 60  0000 C CNN
-	1    14050 6100
-	1    0    0    -1
-$EndComp
-$Comp
 L CONN_1 P8
 U 1 1 53055559
@@
 	1    0    0    -1
 $EndComp
-$Comp
-L CONN_1 P11
-U 1 1 53055586
-P 14050 7300
-F 0 "P11" H 14130 7300 40  0000 L CNN
-F 1 "CONN_1" H 14050 7355 30  0001 C CNN
-F 2 "" H 14050 7300 60  0000 C CNN
-F 3 "" H 14050 7300 60  0000 C CNN
-	1    14050 7300
-	1    0    0    -1
-$EndComp
-$Comp
-L CONN_1 P13
-U 1 1 53055595
-P 14100 7600
-F 0 "P13" H 14180 7600 40  0000 L CNN
-F 1 "CONN_1" H 14100 7655 30  0001 C CNN
-F 2 "" H 14100 7600 60  0000 C CNN
-F 3 "" H 14100 7600 60  0000 C CNN
-	1    14100 7600
-	1    0    0    -1
-$EndComp
-NoConn ~ 13950 5750
-NoConn ~ 13900 6100
 NoConn ~ 13900 6400
 NoConn ~ 13900 6750
 NoConn ~ 13900 6950
-NoConn ~ 13900 7300
-NoConn ~ 13950 7600
 Wire Wire Line
 	8310 1165 8310 1215
@@
 	0    1    1    0
 $EndComp
+$Comp
+L CONN_1 P7
+U 1 1 543FD10D
+P 14050 6250
+F 0 "P7" H 14130 6250 40  0000 L CNN
+F 1 "CONN_1" H 14050 6305 30  0001 C CNN
+F 2 "" H 14050 6250 60  0000 C CNN
+F 3 "" H 14050 6250 60  0000 C CNN
+	1    14050 6250
+	1    0    0    -1
+$EndComp
+NoConn ~ 13900 6250
 $EndSCHEMATC

Commit message: silkscreen new
Parts:
- D10, D6, D8: value LED -> LED VERDE
- D11, D7, D9: value LED -> LED ROJO
- R1, R13, R15, R17, R18, R3: value 1k -> 4.02k
- R27: value R -> 4.02k
- R28: value R -> 1k
- R6: value 3.9k -> 18k
Changed lines of the file:
@@
 Sheet 1 1
 Title ""
-Date "16 oct 2014"
+Date "26 jan 2015"
 Rev ""
 Comp ""
@@
 P 11370 580
 F 0 "R1" V 11450 580 40  0000 C CNN
-F 1 "1k" V 11377 581 40  0000 C CNN
+F 1 "4.02k" V 11377 581 40  0000 C CNN
 F 2 "~" V 11300 580 30  0000 C CNN
 F 3 "~" H 11370 580 30  0000 C CNN
@@
 P 11370 845
 F 0 "R3" V 11450 845 40  0000 C CNN
-F 1 "1k" V 11377 846 40  0000 C CNN
+F 1 "4.02k" V 11377 846 40  0000 C CNN
 F 2 "~" V 11300 845 30  0000 C CNN
 F 3 "~" H 11370 845 30  0000 C CNN
@@
 P 10995 3655
 F 0 "R13" V 11075 3655 40  0000 C CNN
-F 1 "1k" V 11002 3656 40  0000 C CNN
+F 1 "4.02k" V 11002 3656 40  0000 C CNN
 F 2 "~" V 10925 3655 30  0000 C CNN
 F 3 "~" H 10995 3655 30  0000 C CNN
@@
 P 10995 3920
 F 0 "R15" V 11075 3920 40  0000 C CNN
-F 1 "1k" V 11002 3921 40  0000 C CNN
+F 1 "4.02k" V 11002 3921 40  0000 C CNN
 F 2 "~" V 10925 3920 30  0000 C CNN
 F 3 "~" H 10995 3920 30  0000 C CNN
@@
 P 10885 5070
 F 0 "R17" V 10965 5070 40  0000 C CNN
-F 1 "1k" V 10892 5071 40  0000 C CNN
+F 1 "4.02k" V 10892 5071 40  0000 C CNN
 F 2 "~" V 10815 5070 30  0000 C CNN
 F 3 "~" H 10885 5070 30  0000 C CNN
@@
 P 10885 5335
 F 0 "R18" V 10965 5335 40  0000 C CNN
-F 1 "1k" V 10892 5336 40  0000 C CNN
+F 1 "4.02k" V 10892 5336 40  0000 C CNN
 F 2 "~" V 10815 5335 30  0000 C CNN
 F 3 "~" H 10885 5335 30  0000 C CNN
@@
 P 2370 -225
 F 0 "R27" V 2450 -225 40  0000 C CNN
-F 1 "R" V 2377 -224 40  0000 C CNN
+F 1 "4.02k" V 2377 -224 40  0000 C CNN
 F 2 "~" V 2300 -225 30  0000 C CNN
 F 3 "~" H 2370 -225 30  0000 C CNN
@@
 P 3185 -5
 F 0 "R28" V 3265 -5  40  0000 C CNN
-F 1 "R" V 3192 -4  40  0000 C CNN
+F 1 "1k" V 3192 -4  40  0000 C CNN
 F 2 "~" V 3115 -5  30  0000 C CNN
 F 3 "~" H 3185 -5  30  0000 C CNN
@@
 P 10450 500
 F 0 "D10" H 10450 600 50  0000 C CNN
-F 1 "LED" H 10450 400 50  0000 C CNN
+F 1 "LED VERDE" H 10450 400 50  0000 C CNN
 F 2 "~" H 10450 500 60  0000 C CNN
 F 3 "~" H 10450 500 60  0000 C CNN
@@
 P 10450 800
 F 0 "D11" H 10450 900 50  0000 C CNN
-F 1 "LED" H 10450 700 50  0000 C CNN
+F 1 "LED ROJO" H 10450 700 50  0000 C CNN
 F 2 "~" H 10450 800 60  0000 C CNN
 F 3 "~" H 10450 800 60  0000 C CNN
@@
 P 10090 3640
 F 0 "D8" H 10090 3740 50  0000 C CNN
-F 1 "LED" H 10090 3540 50  0000 C CNN
+F 1 "LED VERDE" H 10090 3540 50  0000 C CNN
 F 2 "~" H 10090 3640 60  0000 C CNN
 F 3 "~" H 10090 3640 60  0000 C CNN
@@
 P 10090 3925
 F 0 "D9" H 10090 4025 50  0000 C CNN
-F 1 "LED" H 10090 3825 50  0000 C CNN
+F 1 "LED ROJO" H 10090 3825 50  0000 C CNN
 F 2 "~" H 10090 3925 60  0000 C CNN
 F 3 "~" H 10090 3925 60  0000 C CNN
@@
 P 9990 5040
 F 0 "D6" H 9990 5140 50  0000 C CNN
-F 1 "LED" H 9990 4940 50  0000 C CNN
+F 1 "LED VERDE" H 9990 4940 50  0000 C CNN
 F 2 "~" H 9990 5040 60  0000 C CNN
 F 3 "~" H 9990 5040 60  0000 C CNN
@@
 P 9995 5415
 F 0 "D7" H 9995 5515 50  0000 C CNN
-F 1 "LED" H 9995 5315 50  0000 C CNN
+F 1 "LED ROJO" H 9995 5315 50  0000 C CNN
 F 2 "~" H 9995 5415 60  0000 C CNN
 F 3 "~" H 9995 5415 60  0000 C CNN
@@
 P 9840 2630
 F 0 "R6" V 9920 2630 40  0000 C CNN
-F 1 "3.9k" V 9847 2631 40  0000 C CNN
+F 1 "18k" V 9847 2631 40  0000 C CNN
 F 2 "~" V 9770 2630 30  0000 C CNN
 F 3 "~" H 9840 2630 30  0000 C CNN
