File: trabajo/kicad/AD2S1210/AD2S1210_AD8662.kicad_pcb (KiCad board)
At the start: 2 copper layers, 75 parts, among them IC1 AD8662, K1 JP_1, K2 V_control, K3 Power, P1 conn_stm32f4, P2 AOUT, P3 conn_motor_control, P4 JP_2, P5 JP_3, Q1 RECOM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

Commit message: new file gerber PCB Three-phase bridge
Parts:
- removed G***: LOGO, LOGO
- moved Drill2 26.5 mm to (92.2, 32.9)
- moved Drill3 22.0 mm to (62.5, 99.5)
- moved Drill4 8.90 mm to (117.8, 99.6)
- moved Drill1 8.33 mm to (45.3, 32.5)
Other:
- board outline added: 93 x 78.7 mm
- net class Default: clearance 0.254 -> 0.1524
- rule trace_clearance: 0.254 -> 0.1524
- board text added: "ARCOS-Lab Open-COROCO Resolver-board Rev-0.1 2014-10-20"
- board text removed: "ARCOS-LAB"
- board text removed: "bottom"
- board text removed: "top"

Commit message: reduccion de resolver
Changed lines of the file:
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@@
     (links 200)
     (no_connects 2)
-    (area 27.8384 26.594599 125.825721 105.411741)
+    (area 32.677899 26.594599 125.825721 105.411741)
     (thickness 1.6)
     (drawings 10)
@@
   )
   (layers
-    (15 F.Cu signal hide)
-    (0 B.Cu signal hide)
+    (15 F.Cu signal)
+    (0 B.Cu signal)
     (16 B.Adhes user hide)
     (17 F.Adhes user hide)
     (18 B.Paste user hide)
     (19 F.Paste user hide)
-    (20 B.SilkS user hide)
-    (21 F.SilkS user hide)
+    (20 B.SilkS user)
+    (21 F.SilkS user)
     (22 B.Mask user hide)
     (23 F.Mask user hide)
-    (28 Edge.Cuts user hide)
+    (28 Edge.Cuts user)
   )
   (setup
@@
     (pad_to_mask_clearance 0)
     (aux_axis_origin 220.98 44.45)
-    (visible_elements FFFFF301)
+    (visible_elements FFFFF379)
     (pcbplotparams
       (layerselection 284196865)
@@
       (effects (font (size 1 1) (thickness 0.15)))
     )
-    (fp_text value RECOM (at -0.635 -5.08 270) (layer F.SilkS)
+    (fp_text value RECOM (at 5.715 -5.5372 270) (layer F.SilkS)
       (effects (font (size 1 1) (thickness 0.15)))
     )
@@
     (descr "Connecteur 3 pins")
     (tags "CONN DEV")
-    (fp_text reference K2 (at 0.254 -2.159 180) (layer F.SilkS)
+    (fp_text reference K2 (at -0.27432 2.02184 180) (layer F.SilkS)
       (effects (font (size 1.016 1.016) (thickness 0.1524)))
     )
@@
       (effects (font (size 1.016 1.016) (thickness 0.1524)))
     )
-    (fp_text value JP_1 (at 0 -2.159 180) (layer F.SilkS) hide
+    (fp_text value JP_1 (at 5.4229 0.5588 180) (layer F.SilkS) hide
       (effects (font (size 1.016 1.016) (thickness 0.1524)))
     )
@@
   (module LQFP48 (layer F.Cu)
     (at 82.55 83.693 270)
-    (fp_text reference AD1 (at 4.572 5.207 360) (layer F.SilkS)
+    (fp_text reference AD1 (at 2.5146 1.7272 360) (layer F.SilkS)
       (effects (font (size 1.27 1.27) (thickness 0.2)))
     )
-    (fp_text value AD2S1210 (at 0 -0.635 270) (layer F.SilkS)
-      (effects (font (size 1.27 1.27) (thickness 0.2)))
+    (fp_text value AD2S1210 (at 0.17526 -1.24714 270) (layer F.SilkS)
+      (effects (font (size 1.27 0.762) (thickness 0.1905)))
     )
     (fp_line (start -3.5 3.5) (end -3.5 3.5) (layer F.SilkS) (width 0.2))
@@
       (effects (font (size 1.016 1.016) (thickness 0.27432)))
     )
-    (fp_text value conn_stm32f4 (at 1.016 38.1) (layer F.SilkS)
+    (fp_text value conn_stm32f4 (at 1.3462 0.00762 90) (layer F.SilkS)
       (effects (font (size 1.016 1.016) (thickness 0.2032)))
     )
@@
       (effects (font (size 1.016 1.016) (thickness 0.27432)))
     )
-    (fp_text value conn_motor_control (at 1.016 38.1) (layer F.SilkS)
+    (fp_text value conn_motor_control (at 1.05664 -0.01016 90) (layer F.SilkS)
       (effects (font (size 1.016 1.016) (thickness 0.2032)))
     )

Commit message: cambio de valores errones
Parts:
- R17, R27: value 13.6k -> 13.3k
Changed lines of the file:
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@@
       (effects (font (size 0.635 0.635) (thickness 0.127)))
     )
-    (fp_text value 13.6k (at 0 0 90) (layer F.SilkS) hide
+    (fp_text value 13.3k (at 0 0 90) (layer F.SilkS) hide
       (effects (font (size 0.635 0.635) (thickness 0.127)))
     )
@@
       (effects (font (size 0.635 0.635) (thickness 0.127)))
     )
-    (fp_text value 13.6k (at 0 0 270) (layer F.SilkS) hide
-      (effects (font (size 0.635 0.635) (thickness 0.127)))
-    )
+    (fp_text value 13.3k (at 0 0 270) (layer F.SilkS) hide
+      (effects (font (size 0.635 0.635) (thickness 0.127)))
+    )

Commit message: resolver kicad pcb: added vout
Parts:
- K2: value V_control -> V_out
Changed lines of the file:
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@@
-(kicad_pcb (version 3) (host pcbnew "(22-Jun-2014 BZR 4027)-stable")
+(kicad_pcb (version 3) (host pcbnew "(25-Oct-2014 BZR 4029)-stable")
   (general
     (links 200)
@@
       (effects (font (size 1.016 1.016) (thickness 0.1524)))
     )
-    (fp_text value V_control (at 0 -2.159 180) (layer F.SilkS) hide
+    (fp_text value V_out (at 0 -2.159 180) (layer F.SilkS)
       (effects (font (size 1.016 1.016) (thickness 0.1524)))
     )
