File: resolver_board/kicad/AD2S1210/AD2S1210_AD8662.kicad_pcb (KiCad board)
At the start: 2 copper layers, 93 x 78.7 mm, 74 parts, among them IC1 AD8662, K1 JP_1, K2 V_control, K3 Power, P1 conn_stm32f4, P2 AOUT, P3 conn_motor_control, P4 JP_2, P5 JP_3, Q1 RECOM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

Commit message: voltage divider added to the resolver_board
Parts:
- added R28: 2.66 K, SM0805, F.Cu at (94.8, 40.7)
- added R29: 2.66 K, SM0805, F.Cu at (87.1, 40.7)
- added R30: 2.66 K, SM0805, F.Cu at (91.0, 40.7)
- added R31: 2.66 K, SM0805, F.Cu at (84.2, 40.7)
Connections:
- P2 pad 1: /OUT_EXC -> (no net)
- P2 pad 2: /OUT_~EXC -> (no net)
Routing:
- net /SINLO: track 71.0 -> 98.4 mm
- net /COSLO: track 59.9 -> 80.2 mm
- net +5V: track 103.2 -> 110.2 mm
- net GND: track 636.7 -> 642.3 mm
